Commit message: intento_1_camara_gps

File: src/vtol_tiltrotor_description/urdf/gazebo_fortress.xacro (robot description, xacro)
@@ -188,4 +188,30 @@
     </plugin>
   </gazebo>
+  <!-- ======================== DEPTH CAMERA + GPS ======================== -->
+  <gazebo reference="depth_camera_link">
+    <sensor name="depth_camera" type="depth_camera">
+      <always_on>1</always_on>
+      <update_rate>10</update_rate>
+      <topic>/${ns}/depth_camera</topic>
+      <ignition_frame_id>depth_camera_link</ignition_frame_id>
+      <camera>
+        <horizontal_fov>1.047</horizontal_fov>
+        <image>
+          <width>320</width>
+          <height>240</height>
+          <format>R_FLOAT32</format>
+        </image>
+        <clip><near>0.2</near><far>30</far></clip>
+      </camera>
+    </sensor>
+  </gazebo>
+  <gazebo reference="gps_link">
+    <sensor name="gps" type="navsat">
+      <always_on>1</always_on>
+      <update_rate>5</update_rate>
+      <topic>/${ns}/navsat</topic>
+      <ignition_frame_id>gps_link</ignition_frame_id>
+    </sensor>
+  </gazebo>
   <!-- ============================= MATERIALS ============================ -->
   <xacro:macro name="gz_color" params="link r g b">

File: src/vtol_tiltrotor_description/urdf/vtol_tiltrotor.urdf.xacro (robot description, xacro)
@@ -201,4 +201,15 @@
     <origin xyz="0.10 0 0.01"/>
   </joint>
+  <!-- ========================= DEPTH CAMERA + GPS ======================= -->
+  <link name="depth_camera_link"/>
+  <joint name="depth_camera_joint" type="fixed">
+    <parent link="base_link"/><child link="depth_camera_link"/>
+    <origin xyz="0.64 0 0" rpy="0 0 0"/>   <!-- justo delante de la esfera de la nariz -->
+  </joint>
+  <link name="gps_link"/>
+  <joint name="gps_joint" type="fixed">
+    <parent link="base_link"/><child link="gps_link"/>
+    <origin xyz="0.20 0 0.10"/>            <!-- sobre el pod -->
+  </joint>
   <!-- ============================== WING =============================== -->
   <!-- Link frame = half-panel aerodynamic centre, so LiftDrag <cp> = 0 0 0 -->
